Commit message: fix(so101): implement hardware homing offset and physical constant scaling
Signed-off-by: XiaoqiangWu <wuxiaoqiang.rtos@huawei.com>

File: robot_description/urdf/lerobot/so101/so101_base.xacro (robot description, xacro)
@@ -345,6 +345,6 @@
 		<child link="jaw" />
 		<axis xyz="0 0 1" />
-		<!-- calibrated limits: raw(2041,3457) home(2749) = (-1.0858,+1.0858) rad -->
-		<limit effort="10" velocity="10" lower="-1.0858" upper="1.0858"/>
+		<!-- Gripper joint: 0.0 = closed, 1.0 = open (similar to SO-ARM100) -->
+		<limit effort="10" velocity="10" lower="0.0" upper="1.0"/>
 	</joint>
 	<transmission name="6_trans">
@@ -420,5 +420,5 @@
 		<child link="upper_arm" />
 		<axis xyz="0 0 1" />
-		<limit effort="10" velocity="10" lower="-1.74533" upper="1.74533" />
+		<limit effort="10" velocity="10" lower="-1.92" upper="1.92" />
 	</joint>
 	<transmission name="2_trans">

File: robot_description/urdf/lerobot/so101/so101_ros2_control.xacro (robot description, xacro)
@@ -29,6 +29,6 @@
         <joint name="2">
             <command_interface name="position">
-                <param name="min">-1.74533</param>
-                <param name="max">1.74533</param>
+                <param name="min">-1.92</param>
+                <param name="max">1.92</param>
             </command_interface>
             <state_interface name="position" />
@@ -61,6 +61,6 @@
         <joint name="6">
             <command_interface name="position">
-                <param name="min">-1.0858</param>
-                <param name="max">1.0858</param>
+                <param name="min">0.0</param>
+                <param name="max">1.0</param>
             </command_interface>
             <state_interface name="position" />
